Commit message: Added iiwa7, new MoveIt

File: kmriiwa_description/urdf/robot/kmriiwa.urdf.xacro (robot description, xacro)
@@ -2,19 +2,22 @@
 <robot name="kmriiwa" xmlns:xacro="http://www.ros.org/wiki/xacro">
   <!-- Import Rviz colors -->
-  <xacro:include filename="$(find kmriiwa_description)/urdf/iiwa14/materials.xacro" />
+  <xacro:include filename="$(find kmriiwa_description)/urdf/iiwa7/materials.xacro" />
   <!--Import the lbr iiwa macro -->
-  <xacro:include filename="$(find kmriiwa_description)/urdf/iiwa14/iiwa14.xacro"/>
+  <xacro:include filename="$(find kmriiwa_description)/urdf/iiwa7/iiwa7.xacro"/>
   <!--Import the kmp200 macro -->
   <xacro:include filename="$(find kmriiwa_description)/urdf/kmp200/kmp200.xacro"/>
+  <!-- Import the gripper -->
+  <xacro:property name="body_color" value="Gazebo/Silver" />
+  <xacro:include filename="$(find gripkit_cr_plus_l_bb_description)/urdf/gripkit_cr_plus_l_bb.xacro" />
   <xacro:property name="arm_base_flange_x_pos" value="0.363" />
   <xacro:property name="arm_base_flange_y_pos" value="-0.184" />
   <xacro:property name="arm_base_flange_z_pos" value="-0.01" />
   <xacro:property name="arm_base_flange_yew" value="-1.5708" />
-  <xacro:property name="riser_flange_height" value="0.26" />
+  <xacro:property name="riser_flange_height" value="0.0" />
   <xacro:property name="riser_flange_radius" value="0.121" />
   <xacro:property name="flange_origin_xyz" value="${arm_base_flange_x_pos} ${arm_base_flange_y_pos} ${arm_base_flange_z_pos+riser_flange_height/2}"/>
   <xacro:property name="flange_origin_rpy" value="0 0 ${arm_base_flange_yew}"/>
   <xacro:arg name="robot_name" default="kmriiwa"/>
-  <xacro:arg name="hardware_interface" default="PositionJointInterface"/>
+  <xacro:arg name="hardware_interface" default="EffortJointInterface"/>
   <xacro:arg name="robot_extras" default="$(find kmriiwa_description)/urdf/robot/empty.xacro" />
   <!--kmp200-->
@@ -42,8 +45,15 @@
   </link>
   <!--iiwa-->
-  <xacro:iiwa14 hardware_interface="$(arg hardware_interface)" robot_name="$(arg robot_name)" parent="$(arg robot_name)_riser_flange_link">
+  <xacro:iiwa7 hardware_interface="PositionJointInterface" robot_name="$(arg robot_name)" parent="$(arg robot_name)_riser_flange_link">
     <origin xyz="0 0 ${riser_flange_height/2}" rpy="0 0 0" />
-  </xacro:iiwa14>
+  </xacro:iiwa7>
   <!-- Optional custom includes such as grippers, sensors, etc... -->
   <xacro:include filename="$(arg robot_extras)"/>
+  <!-- gripper -->
+  <xacro:gripkit_cr_plus_l_bb />
+  <joint name="Rigid09" type="fixed">
+    <origin xyz="0 0 0.0351" rpy="0 0 0"/>
+    <parent link="$(arg robot_name)_link_7"/>
+    <child link="SF-ISO50-CRG200_Customer"/>
+  </joint>
 </robot>
