Commit message: Gripper control works

File: kmriiwa_moveit/config/kmriiwa.srdf.xacro (robot description, xacro)
@@ -16,5 +16,6 @@
     </group>
     <group name="$(arg robot_name)_endeffector">
-        <link name="$(arg robot_name)_link_ee"/>
+        <joint name="Slider01"/>
+        <joint name="Slider02"/>
     </group>
     <!--GROUP STATES: Purpose: Define a named state for a particular group, in terms of joint values. This is useful to define states like 'folded arms'-->
@@ -36,4 +37,12 @@
         <joint name="$(arg robot_name)_joint_6" value="0.8827"/>
         <joint name="$(arg robot_name)_joint_7" value="0.662003"/>
+    </group_state>
+    <group_state name="open" group="kmriiwa_endeffector">
+        <joint name="Slider01" value="-0.021"/>
+        <joint name="Slider02" value="0.021"/>
+    </group_state>
+    <group_state name="closed" group="kmriiwa_endeffector">
+        <joint name="Slider01" value="0"/>
+        <joint name="Slider02" value="0"/>
     </group_state>
     <xacro:unless value="$(arg no_virtual_joint)">
