Commit message: Figuring out where PID gains are defined

File: gripkit_cr_plus_l_bb_description/urdf/gripkit_cr_plus_l_bb.xacro (robot description, xacro)
@@ -19,5 +19,5 @@
           <mesh filename="package://gripkit_cr_plus_l_bb_description/meshes/SF-ISO50-CRG200_Customer.stl" scale="0.001 0.001 0.001"/>
         </geometry>
-        <material name="silver"/>
+        <material name="Gazebo/Grey"/>
       </visual>
       <collision>
@@ -39,5 +39,5 @@
           <mesh filename="package://gripkit_cr_plus_l_bb_description/meshes/CRG200_body.stl" scale="0.001 0.001 0.001"/>
         </geometry>
-        <material name="silver"/>
+        <material name="Gazebo/Grey"/>
       </visual>
       <collision>
@@ -59,5 +59,5 @@
           <mesh filename="package://gripkit_cr_plus_l_bb_description/meshes/CRG200_base_jaw_1.stl" scale="0.001 0.001 0.001"/>
         </geometry>
-        <material name="silver"/>
+        <material name="Gazebo/Grey"/>
       </visual>
       <collision>
@@ -79,5 +79,5 @@
           <mesh filename="package://gripkit_cr_plus_l_bb_description/meshes/CRG200_base_jaw_2.stl" scale="0.001 0.001 0.001"/>
         </geometry>
-        <material name="silver"/>
+        <material name="Gazebo/Grey"/>
       </visual>
       <collision>
@@ -99,5 +99,5 @@
           <mesh filename="package://gripkit_cr_plus_l_bb_description/meshes/CRG200_top_cover.stl" scale="0.001 0.001 0.001"/>
         </geometry>
-        <material name="silver"/>
+        <material name="Gazebo/Grey"/>
       </visual>
       <collision>
@@ -119,5 +119,5 @@
           <mesh filename="package://gripkit_cr_plus_l_bb_description/meshes/ISO_4762_-_M4_x_12ISO_1.stl" scale="0.001 0.001 0.001"/>
         </geometry>
-        <material name="silver"/>
+        <material name="Gazebo/Grey"/>
       </visual>
       <collision>
@@ -139,5 +139,5 @@
           <mesh filename="package://gripkit_cr_plus_l_bb_description/meshes/ISO_4762_-_M4_x_12ISO_2.stl" scale="0.001 0.001 0.001"/>
         </geometry>
-        <material name="silver"/>
+        <material name="Gazebo/Grey"/>
       </visual>
       <collision>
@@ -159,5 +159,5 @@
           <mesh filename="package://gripkit_cr_plus_l_bb_description/meshes/ISO_4762_-_M4_x_12ISO_3.stl" scale="0.001 0.001 0.001"/>
         </geometry>
-        <material name="silver"/>
+        <material name="Gazebo/Grey"/>
       </visual>
       <collision>
@@ -179,5 +179,5 @@
           <mesh filename="package://gripkit_cr_plus_l_bb_description/meshes/ISO_4762_-_M4_x_12ISO_4.stl" scale="0.001 0.001 0.001"/>
         </geometry>
-        <material name="silver"/>
+        <material name="Gazebo/Grey"/>
       </visual>
       <collision>
@@ -199,5 +199,5 @@
           <mesh filename="package://gripkit_cr_plus_l_bb_description/meshes/BE_20-030_CUSTOMER_v1_1.stl" scale="0.001 0.001 0.001"/>
         </geometry>
-        <material name="silver"/>
+        <material name="Gazebo/Grey"/>
       </visual>
       <collision>
@@ -219,5 +219,5 @@
           <mesh filename="package://gripkit_cr_plus_l_bb_description/meshes/BE_20-030_CUSTOMER_v1_2.stl" scale="0.001 0.001 0.001"/>
         </geometry>
-        <material name="silver"/>
+        <material name="Gazebo/Grey"/>
       </visual>
       <collision>
@@ -239,5 +239,5 @@
           <mesh filename="package://gripkit_cr_plus_l_bb_description/meshes/AC_20-025_CUSTOMER_v1_1.stl" scale="0.001 0.001 0.001"/>
         </geometry>
-        <material name="silver"/>
+        <material name="Gazebo/Grey"/>
       </visual>
       <collision>
@@ -259,5 +259,5 @@
           <mesh filename="package://gripkit_cr_plus_l_bb_description/meshes/AC_20-025_CUSTOMER_v1_2.stl" scale="0.001 0.001 0.001"/>
         </geometry>
-        <material name="silver"/>
+        <material name="Gazebo/Grey"/>
       </visual>
       <collision>
@@ -279,5 +279,5 @@
           <mesh filename="package://gripkit_cr_plus_l_bb_description/meshes/FT_20-CR_CUSTOMER_v1_1.stl" scale="0.001 0.001 0.001"/>
         </geometry>
-        <material name="silver"/>
+        <material name="Gazebo/Grey"/>
       </visual>
       <collision>
@@ -299,5 +299,5 @@
           <mesh filename="package://gripkit_cr_plus_l_bb_description/meshes/FT_20-CR_CUSTOMER_v1_2.stl" scale="0.001 0.001 0.001"/>
         </geometry>
-        <material name="silver"/>
+        <material name="Gazebo/Grey"/>
       </visual>
       <collision>

File: kmriiwa_description/urdf/kmp200/kmp200.gazebo.xacro (robot description, xacro)
@@ -38,5 +38,5 @@
         <sensor name="sensor_B1" type="ray">
             <always_on>true</always_on>
-            <visualize>true</visualize>
+            <visualize>false</visualize>
             <update_rate>10</update_rate>
             <ray>
@@ -71,5 +71,5 @@
         <sensor name="sensor_B4" type="ray">
             <always_on>true</always_on>
-            <visualize>true</visualize>
+            <visualize>false</visualize>
             <update_rate>10</update_rate>
             <ray>
